File: TreeOrnamentV2.kicad_pcb (KiCad board)
At the start: 2 copper layers, 50.8 x 73.7 mm, 25 parts, among them SW1 SW_SPDT, U1 ATTINY85-20SU

Commit message: Fix Switch Track
Move track from switch to power ATTiny so it doesn't cross VCC pad of battery holder
Routing:
- net Net-(SW1-Pad1): track 42.5 -> 44.9 mm
Other:
- board text added: "29-04-2017 brd #02 Rev3"
- board text removed: "29-04-2017 brd #02 Rev2"
Changed lines of the file:
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@@
-(kicad_pcb (version 20170123) (host pcbnew no-vcs-found-0633d90~59~ubuntu16.04.1)
+(kicad_pcb (version 20170123) (host pcbnew no-vcs-found-d41af7d~59~ubuntu16.04.1)
   (general
     (thickness 1.6)
     (drawings 95)
-    (tracks 227)
+    (tracks 226)
     (zones 0)
     (modules 25)
@@
   (gr_line (start 144.78 116.84) (end 137.16 116.84) (layer Edge.Cuts) (width 0.15))
   (gr_line (start 139.7 114.3) (end 144.78 116.84) (layer Edge.Cuts) (width 0.15))
-  (gr_text "29-04-2017\nbrd #02 Rev2" (at 120.396 108.458) (layer B.SilkS)
+  (gr_text "29-04-2017\nbrd #02 Rev3" (at 120.396 108.458) (layer B.SilkS)
     (effects (font (size 0.75 0.75) (thickness 0.125)) (justify mirror))
   )
@@
   (segment (start 139.606 99.6622) (end 140.3803 100.4365) (width 0.2032) (layer F.Cu) (net 17))
   (segment (start 140.3803 100.4365) (end 141.0335 100.4365) (width 0.2032) (layer F.Cu) (net 17) (status 20))
+  (segment (start 119.928 103.954) (end 120.7312 103.954) (width 0.2032) (layer B.Cu) (net 19))
+  (segment (start 133.743602 98.269756) (end 134.223358 97.79) (width 0.2032) (layer B.Cu) (net 19))
+  (segment (start 120.7312 103.954) (end 124.3552 100.33) (width 0.2032) (layer B.Cu) (net 19))
+  (segment (start 144.526 100.965) (end 146.685 100.965) (width 0.2032) (layer B.Cu) (net 19))
+  (segment (start 124.3552 100.33) (end 133.743602 100.33) (width 0.2032) (layer B.Cu) (net 19))
+  (segment (start 133.743602 100.33) (end 133.743602 98.269756) (width 0.2032) (layer B.Cu) (net 19))
+  (segment (start 134.223358 97.79) (end 141.351 97.79) (width 0.2032) (layer B.Cu) (net 19))
+  (segment (start 141.351 97.79) (end 144.526 100.965) (width 0.2032) (layer B.Cu) (net 19))
   (segment (start 146.685 100.00925) (end 142.328899 95.653149) (width 0.2032) (layer F.Cu) (net 19))
   (segment (start 146.685 100.965) (end 146.685 100.00925) (width 0.2032) (layer F.Cu) (net 19))
@@
   (via (at 142.621 92.964) (size 0.6858) (drill 0.3302) (layers F.Cu B.Cu) (net 19))
   (via (at 141.986 94.869) (size 0.6858) (drill 0.3302) (layers F.Cu B.Cu) (net 19))
-  (segment (start 142.748 99.187) (end 144.526 100.965) (width 0.2032) (layer B.Cu) (net 19))
-  (segment (start 144.526 100.965) (end 146.685 100.965) (width 0.2032) (layer B.Cu) (net 19))
   (via (at 146.685 100.965) (size 0.6858) (drill 0.3302) (layers F.Cu B.Cu) (net 19))
-  (segment (start 135.001 99.187) (end 142.748 99.187) (width 0.2032) (layer B.Cu) (net 19))
-  (segment (start 133.800801 100.387199) (end 135.001 99.187) (width 0.2032) (layer B.Cu) (net 19))
-  (segment (start 133.165801 100.387199) (end 133.800801 100.387199) (width 0.2032) (layer B.Cu) (net 19))
-  (segment (start 124.2282 100.457) (end 124.298001 100.387199) (width 0.2032) (layer B.Cu) (net 19))
-  (segment (start 124.298001 100.387199) (end 133.165801 100.387199) (width 0.2032) (layer B.Cu) (net 19))
-  (segment (start 119.928 103.954) (end 120.7312 103.954) (width 0.2032) (layer B.Cu) (net 19))
-  (segment (start 120.7312 103.954) (end 124.2282 100.457) (width 0.2032) (layer B.Cu) (net 19))
   (zone (net 8) (net_name /VCC) (layer B.Cu) (hatch edge 0.508)
     (connect_pads (clearance 0.508))
