File: TreeOrnamentV2.sch (KiCad schematic (older format))
At the start: 23 parts, among them SW1 SW_SPDT, U1 ATTINY85-20SU

Commit message: KiCad Symbol Update
Update to how KiCad uses sybols
Parts:
- removed BT1: Battery_Cell, Battery_Holders:Keystone_3002_1x2032-CoinCell, symbol Battery_Cell
- added BT1: Battery_Cell, symbol device:Battery_Cell
- D10, D11, D12, D2, D3, D4, D5, D6, D8, D9: symbol LED -> device:LED
- R10, R11, R12, R2, R3, R4, R5, R6, R8, R9: symbol R -> device:R
- SW1: symbol SW_SPDT -> Switch:SW_SPDT
- U1: symbol ATTINY85-20SU -> atmel:ATTINY85-20SU
Connections:
- net GND: now also BT1.2 (-)
- net VCC: now also BT1.1 (+)
Changed lines of the file:
@@
-EESchema Schematic File Version 2
-LIBS:power
-LIBS:device
-LIBS:transistors
-LIBS:conn
-LIBS:linear
-LIBS:regul
-LIBS:74xx
-LIBS:cmos4000
-LIBS:adc-dac
-LIBS:memory
-LIBS:xilinx
-LIBS:microcontrollers
-LIBS:dsp
-LIBS:microchip
-LIBS:analog_switches
-LIBS:motorola
-LIBS:texas
-LIBS:intel
-LIBS:audio
-LIBS:interface
-LIBS:digital-audio
-LIBS:philips
-LIBS:display
-LIBS:cypress
-LIBS:siliconi
-LIBS:opto
-LIBS:atmel
-LIBS:contrib
-LIBS:valves
-LIBS:custom
-LIBS:switches
+EESchema Schematic File Version 4
 LIBS:TreeOrnamentV2-cache
 EELAYER 26 0
@@
 $EndDescr
 $Comp
-L Battery_Cell BT1
-U 1 1 58B89C6D
-P 1325 3450
-F 0 "BT1" H 1425 3550 50  0000 L CNN
-F 1 "Battery_Cell" H 1425 3450 50  0000 L CNN
-F 2 "Battery_Holders:Keystone_3002_1x2032-CoinCell" V 1325 3510 50  0001 C CNN
-F 3 "" V 1325 3510 50  0001 C CNN
-	1    1325 3450
-	1    0    0    -1
-$EndComp
-$Comp
-L GND #PWR01
+L TreeOrnamentV2-rescue:GND-RESCUE-TreeOrnamentV2 #PWR01
 U 1 1 58B89D01
 P 1325 4000
@@
 VCC
 $Comp
-L PWR_FLAG #FLG02
-U 1 1 58B8F65A
-P 1325 3875
-F 0 "#FLG02" H 1325 3950 50  0001 C CNN
-F 1 "PWR_FLAG" H 1325 4025 50  0000 C CNN
-F 2 "" H 1325 3875 50  0001 C CNN
-F 3 "" H 1325 3875 50  0001 C CNN
-	1    1325 3875
-	0    -1   -1   0
-$EndComp
-$Comp
-L SW_SPDT SW1
+L Switch:SW_SPDT SW1
 U 1 1 58C42CFA
 P 2775 2625
@@
 VCC
 $Comp
-L ATTINY85-20SU U1
+L atmel:ATTINY85-20SU U1
 U 1 1 58CB39BC
 P 5100 3425
@@
 $EndComp
 $Comp
-L GND #PWR03
-U 1 1 58CB3AC1
-P 3750 3175
-F 0 "#PWR03" H 3750 2925 50  0001 C CNN
-F 1 "GND" V 3755 3047 50  0000 R CNN
-F 2 "" H 3750 3175 50  0001 C CNN
-F 3 "" H 3750 3175 50  0001 C CNN
-	1    3750 3175
-	0    1    1    0
-$EndComp
-$Comp
-L LED D2
+L device:LED D2
 U 1 1 58CB428C
 P 7775 3850
@@
 $EndComp
 $Comp
-L LED D8
+L device:LED D8
 U 1 1 58CB43C2
 P 8325 3850
@@
 $EndComp
 $Comp
-L R R2
+L device:R R2
 U 1 1 58CB44CF
 P 7775 3550
@@
 $EndComp
 $Comp
-L LED D3
+L device:LED D3
 U 1 1 58CB4A28
 P 7775 4825
@@
 $EndComp
 $Comp
-L LED D9
+L device:LED D9
 U 1 1 58CB4A2E
 P 8325 4825
@@
 $EndComp
 $Comp
-L R R3
+L device:R R3
 U 1 1 58CB4A34
 P 7775 4525
@@
 $EndComp
 $Comp
-L LED D4
+L device:LED D4
 U 1 1 58CB4A40
 P 10325 2850
@@
 $EndComp
 $Comp
-L LED D10
+L device:LED D10
 U 1 1 58CB4A46
 P 10875 2850
@@
 $EndComp
 $Comp
-L R R4
+L device:R R4
 U 1 1 58CB4A4E
 P 10325 2550
@@
 $EndComp
 $Comp
-L LED D5
+L device:LED D5
 U 1 1 58CB4F2B
 P 10325 3850
@@
 $EndComp
 $Comp
-L LED D11
+L device:LED D11
 U 1 1 58CB4F31
 P 10875 3850
@@
 $EndComp
 $Comp
-L R R5
+L device:R R5
 U 1 1 58CB4F37
 P 10325 3550
@@
 $EndComp
 $Comp
-L LED D6
+L device:LED D6
 U 1 1 58CB4F43
 P 10325 4825
@@
 $EndComp
 $Comp
-L LED D12
+L device:LED D12
 U 1 1 58CB4F49
 P 10875 4825
@@
 $EndComp
 $Comp
-L R R6
+L device:R R6
 U 1 1 58CB4F51
 P 10325 4525
@@
 $EndComp
 $Comp
-L GND #PWR04
+L power:GND #PWR04
 U 1 1 58D5F707
 P 8825 4000
@@
 Pin2
 $Comp
-L GND #PWR05
+L power:GND #PWR05
 U 1 1 58D5FE02
 P 8825 4975
@@
 Pin3
 $Comp
-L GND #PWR06
+L power:GND #PWR06
 U 1 1 58D5FE25
 P 11375 3000
@@
 Pin4
 $Comp
-L GND #PWR07
+L power:GND #PWR07
 U 1 1 58D60118
 P 11375 4000
@@
 Pin5
 $Comp
-L GND #PWR08
+L power:GND #PWR08
 U 1 1 58D60B64
 P 11375 4975
@@
 Pin6
 $Comp
-L R R8
+L device:R R8
 U 1 1 58D6513F
 P 8325 3550
@@
 $EndComp
 $Comp
-L R R9
+L device:R R9
 U 1 1 58D65D55
 P 8325 4525
@@
 $EndComp
 $Comp
-L R R10
+L device:R R10
 U 1 1 58D66545
 P 10875 2550
@@
 Wire Wire Line
 	1325 3550 1325 4000
-Connection ~ 1325 3875
 Wire Wire Line
 	2375 2625 2575 2625
@@
 Connection ~ 10325 3375
 $Comp
-L R R11
+L device:R R11
 U 1 1 58D66B3C
 P 10875 3550
@@
 Connection ~ 10325 4355
 $Comp
-L R R12
+L device:R R12
 U 1 1 58D670E4
 P 10875 4525
@@
 Wire Wire Line
 	10875 4355 10875 4375
+$Comp
+L power:GND #PWR02
+U 1 1 5A07A38D
+P 3750 3175
+F 0 "#PWR02" H 3750 2925 50  0001 C CNN
+F 1 "GND" V 3755 3047 50  0000 R CNN
+F 2 "" H 3750 3175 50  0001 C CNN
+F 3 "" H 3750 3175 50  0001 C CNN
+	1    3750 3175
+	0    1    1    0
+$EndComp
+$Comp
+L device:Battery_Cell BT1
+U 1 1 5A07A5E9
+P 1325 3450
+F 0 "BT1" H 1443 3546 50  0000 L CNN
+F 1 "Battery_Cell" H 1443 3455 50  0000 L CNN
+F 2 "" V 1325 3510 50  0001 C CNN
+F 3 "" V 1325 3510 50  0001 C CNN
+	1    1325 3450
+	1    0    0    -1
+$EndComp
 $EndSCHEMATC
